Commit message: Update control configs and cleanup launch files
Removed unused hardware interface and real-world launch file, updated velocity and acceleration limits in control.yaml, and adjusted wheel velocity limits in URDF. Modified Gazebo world object poses, launch parameters, and node topic names for improved simulation and control behavior.

File: urdf/controls/jackal_ros2_control.urdf.xacro (robot description, xacro)
@@ -2,85 +2,41 @@
 <robot xmlns:xacro="http://www.ros.org/wiki/xacro">
   <xacro:macro name="jackal_ros2_control" params="use_gazebo">
-    <xacro:if value="${use_gazebo}">
-      <ros2_control name="GazeboSystem" type="system">
-        <hardware>
-          <plugin>gz_ros2_control/GazeboSimSystem</plugin>
-        </hardware>
-        <!-- Define velocity control for all 4 wheels -->
-        <joint name="front_left_wheel">
-          <command_interface name="velocity">
-            <param name="min">-100</param>
-            <param name="max">100</param>
-          </command_interface>
-          <state_interface name="position"/>
-          <state_interface name="velocity"/>
-        </joint>
-        <joint name="front_right_wheel">
-          <command_interface name="velocity">
-            <param name="min">-100</param>
-            <param name="max">100</param>
-          </command_interface>
-          <state_interface name="position"/>
-          <state_interface name="velocity"/>
-        </joint>
-        <joint name="rear_left_wheel">
-          <command_interface name="velocity">
-            <param name="min">-100</param>
-            <param name="max">100</param>
-          </command_interface>
-          <state_interface name="position"/>
-          <state_interface name="velocity"/>
-        </joint>
-        <joint name="rear_right_wheel">
-          <command_interface name="velocity">
-            <param name="min">-100</param>
-            <param name="max">100</param>
-          </command_interface>
-          <state_interface name="position"/>
-          <state_interface name="velocity"/>
-        </joint>
-      </ros2_control>
-    </xacro:if>
-    <xacro:unless value="${use_gazebo}">
-      <ros2_control name="JackalSystem" type="system">
-        <hardware>
-          <plugin>jackal_base/JackalSystemHardware</plugin>
-        </hardware>
-        <param name="serial_port">/dev/ttyACM0</param>
-        <!-- Define velocity control for all 4 wheels -->
-        <joint name="front_left_wheel">
-          <command_interface name="velocity">
-            <param name="min">-10</param>
-            <param name="max">10</param>
-          </command_interface>
-          <state_interface name="position"/>
-          <state_interface name="velocity"/>
-        </joint>
-        <joint name="front_right_wheel">
-          <command_interface name="velocity">
-            <param name="min">-10</param>
-            <param name="max">10</param>
-          </command_interface>
-          <state_interface name="position"/>
-          <state_interface name="velocity"/>
-        </joint>
-        <joint name="rear_left_wheel">
-          <command_interface name="velocity">
-            <param name="min">-10</param>
-            <param name="max">10</param>
-          </command_interface>
-          <state_interface name="position"/>
-          <state_interface name="velocity"/>
-        </joint>
-        <joint name="rear_right_wheel">
-          <command_interface name="velocity">
-            <param name="min">-10</param>
-            <param name="max">10</param>
-          </command_interface>
-          <state_interface name="position"/>
-          <state_interface name="velocity"/>
-        </joint>
-      </ros2_control>
-    </xacro:unless>
+    <ros2_control name="GazeboSystem" type="system">
+      <hardware>
+        <plugin>gz_ros2_control/GazeboSimSystem</plugin>
+      </hardware>
+      <!-- Define velocity control for all 4 wheels -->
+      <joint name="front_left_wheel">
+        <command_interface name="velocity">
+          <param name="min">-10</param>
+          <param name="max">10</param>
+        </command_interface>               <state_interface name="position"/>
+        <state_interface name="velocity"/>
+      </joint>
+      <joint name="front_right_wheel">
+        <command_interface name="velocity">
+          <param name="min">-10</param>
+          <param name="max">10</param>
+        </command_interface>
+        <state_interface name="position"/>
+        <state_interface name="velocity"/>
+      </joint>
+      <joint name="rear_left_wheel">
+        <command_interface name="velocity">
+          <param name="min">-10</param>
+          <param name="max">10</param>
+        </command_interface>
+        <state_interface name="position"/>
+        <state_interface name="velocity"/>
+     </joint>
+      <joint name="rear_right_wheel">
+        <command_interface name="velocity">
+          <param name="min">-10</param>
+          <param name="max">10</param>
+        </command_interface>               <state_interface name="position"/>
+        <state_interface name="velocity"/>
+      </joint>
+    </ros2_control>
+    <!-- 🔧 Add required transmissions for each wheel -->
   </xacro:macro>
 </robot>
